File: Rochelle_circuit/Rochelle_circuit.kicad_sch (KiCad schematic)
At the start: 16 parts, among them U1 INA125, U2 LM358

Commit message: Changed name of current kicad design, and added Testing code
Parts:
- removed RV2: Linear_Pot, symbol Device:R_Potentiometer_US
- LiquidWire1: value 44-54 -> 5
- R5, R8: value 330k -> 27k
- R6: value 48 -> 120
- RV1: value 10 -> 5
Other:
- note added: "Cutoff Frequency at 60 Hz"
- note removed: "Cutoff Frequency at 50 Hz"
- note removed: "Linear Potentiometer"
- note removed: "Replaced Trimming Potentiometer with an 8.2 Ohm Resistor since the LW sensor currently hooked up to the circuit ranges from like 8 Ohms to 15 Ohms."
Changed lines of the file:
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@@
-	)
-	(rectangle
-		(start 351.79 201.93)
-		(end 383.54 233.68)
-		(stroke
-			(width 0.381)
-			(type solid)
-		)
-		(fill
-			(type none)
-		)
 	)
 	(rectangle
@@
 			(width 0.381)
 			(type solid)
-		)
-		(fill
-			(type none)
-		)
-	)
-	(rectangle
-		(start 64.77 203.2)
-		(end 128.27 212.09)
-		(stroke
-			(width 0)
-			(type default)
 		)
 		(fill
@@
 		)
 	)
-	(text "Replaced Trimming Potentiometer with an 8.2 Ohm Resistor\nsince the LW sensor currently hooked up to the circuit ranges\nfrom like 8 Ohms to 15 Ohms."
-		(exclude_from_sim no)
-		(at 96.774 207.772 0)
-		(effects
-			(font
-				(size 1.27 1.27)
-			)
-		)
-	)
-	(text "Cutoff Frequency at 50 Hz"
+	(text "Cutoff Frequency at 60 Hz"
 		(exclude_from_sim no)
 		(at 286.004 123.19 0)
@@
 		)
 	)
-	(text "Linear Potentiometer"
-		(exclude_from_sim no)
-		(at 367.792 199.39 0)
-		(effects
-			(font
-				(size 1.651 1.651)
-				(thickness 0.2064)
-			)
-		)
-	)
 	(text "Active Low-Pass Filter"
 		(exclude_from_sim no)
@@
 	(wire
 		(pts
-			(xy 363.22 218.44) (xy 363.22 222.25)
-		)
-		(stroke
-			(width 0)
-			(type default)
-		)
-	)
-	(wire
-		(pts
-			(xy 345.44 149.86) (xy 355.6 149.86)
-		)
-		(stroke
-			(width 0)
-			(type default)
-		)
-	)
-	(wire
-		(pts
 			(xy 187.96 88.9) (xy 187.96 124.46)
 		)
@@
 	(wire
 		(pts
-			(xy 359.41 214.63) (xy 345.44 214.63)
-		)
-		(stroke
-			(width 0)
-			(type default)
-		)
-	)
-	(wire
-		(pts
 			(xy 66.04 180.34) (xy 66.04 184.15)
 		)
@@
 	(wire
 		(pts
-			(xy 345.44 214.63) (xy 345.44 149.86)
-		)
-		(stroke
-			(width 0)
-			(type default)
-		)
-	)
-	(wire
-		(pts
 			(xy 66.04 88.9) (xy 66.04 127)
 		)
@@
 	(wire
 		(pts
-			(xy 363.22 187.96) (xy 363.22 210.82)
-		)
-		(stroke
-			(width 0)
-			(type default)
-		)
-	)
-	(wire
-		(pts
 			(xy 132.08 85.09) (xy 132.08 111.76)
 		)
@@
 		(pts
 			(xy 78.74 162.56) (xy 78.74 168.91)
-		)
-		(stroke
-			(width 0)
-			(type default)
-		)
-	)
-	(polyline
-		(pts
-			(xy 78.74 177.8) (xy 81.28 203.2)
 		)
 		(stroke
@@
 			)
 		)
-		(property "Value" "330k"
+		(property "Value" "27k"
 			(at 278.13 146.05 90)
 			(effects
@@
 			)
 		)
-		(property "Value" "44-54"
+		(property "Value" "5"
 			(at 57.15 173.9518 0)
 			(effects
@@
 			)
 		)
-		(property "Value" "10"
+		(property "Value" "5"
 			(at 76.2 173.9899 0)
 			(effects
@@
 			)
 		)
-		(property "Value" "330k"
+		(property "Value" "27k"
 			(at 260.35 146.05 90)
 			(effects
@@
 			)
 		)
-		(property "Value" "48"
+		(property "Value" "120"
 			(at 152.4 166.37 90)
 			(effects
@@
 				(path "/e06ad2b5-2cad-4e7a-b65c-42b4d2c7f012"
 					(reference "#PWR02")
-					(unit 1)
-				)
-			)
-		)
-	)
-	(symbol
-		(lib_id "Device:R_Potentiometer_US")
-		(at 363.22 214.63 180)
-		(unit 1)
-		(exclude_from_sim no)
-		(in_bom yes)
-		(on_board yes)
-		(dnp no)
-		(fields_autoplaced yes)
-		(property "Reference" "RV2"
-			(at 365.76 213.3599 0)
-			(effects
-				(font
-					(size 1.27 1.27)
-				)
-				(justify right)
-			)
-		)
-		(property "Value" "Linear_Pot"
-			(at 365.76 215.8999 0)
-			(effects
-				(font
-					(size 1.27 1.27)
-				)
-				(justify right)
-			)
-		)
-		(property "Footprint" ""
-			(at 363.22 214.63 0)
-			(effects
-				(font
-					(size 1.27 1.27)
-				)
-				(hide yes)
-			)
-		)
-		(property "Datasheet" "~"
-			(at 363.22 214.63 0)
-			(effects
-				(font
-					(size 1.27 1.27)
-				)
-				(hide yes)
-			)
-		)
-		(property "Description" "Potentiometer, US symbol"
-			(at 363.22 214.63 0)
-			(effects
-				(font
-					(size 1.27 1.27)
-				)
-				(hide yes)
-			)
-		)
-		(pin "2"
-		)
-		(pin "1"
-		)
-		(pin "3"
-		)
-		(instances
-			(project ""
-				(path "/e06ad2b5-2cad-4e7a-b65c-42b4d2c7f012"
-					(reference "RV2")
 					(unit 1)
 				)
@@
 					(unit 1)
 				)
-			)
-		)
-	)
-	(symbol
-		(lib_id "power:GND")
-		(at 363.22 222.25 0)
-		(unit 1)
-		(exclude_from_sim no)
-		(in_bom yes)
-		(on_board yes)
-		(dnp no)
-		(property "Reference" "#PWR05"
-			(at 363.22 228.6 0)
-			(effects
-				(font
-					(size 1.27 1.27)
-				)
-				(hide yes)
-			)
-		)
-		(property "Value" "GND"
-			(at 367.538 224.028 0)
-			(effects
-				(font
-					(size 1.27 1.27)
-				)
-			)
-		)
-		(property "Footprint" ""
-			(at 363.22 222.25 0)
-			(effects
-				(font
-					(size 1.27 1.27)
-				)
-				(hide yes)
-			)
-		)
-		(property "Datasheet" ""
-			(at 363.22 222.25 0)
-			(effects
-				(font
-					(size 1.27 1.27)
-				)
-				(hide yes)
-			)
-		)
-		(property "Description" "Power symbol creates a global label with name \"GND\" , ground"
-			(at 363.22 222.25 0)
-			(effects
-				(font
-					(size 1.27 1.27)
-				)
-				(hide yes)
-			)
-		)
-		(pin "1"
-		)
-		(instances
-			(project "Rochelle_circuit"
-				(path "/e06ad2b5-2cad-4e7a-b65c-42b4d2c7f012"
-					(reference "#PWR05")
-					(unit 1)
-				)
